File: _autosave-arduino_pro_mini.sch (KiCad schematic (older format))
At the start: 18 parts, among them J1 Conn_02x03_Odd_Even, J2 Conn_01x10, J3 Conn_01x10, SW1 SW_Push, U1 MIC5205-2.5YM5, U2 ATmega328-AU, Y1 16MHZ

Commit message: first bgr file upload
Parts:
- removed JP1: SolderJumper_2_Bridged, Jumper:SolderJumper-2_P1.3mm_Bridged2Bar_Pad1.0x1.5mm, symbol Jumper:SolderJumper_2_Bridged
Connections:
- net VCC: now also D1.2 (A), U1.5 (OUT)
Changed lines of the file:
@@
 	2650 2500 2750 2500
 Connection ~ 2750 2500
-$Comp
-L Jumper:SolderJumper_2_Bridged JP1
-U 1 1 6071A14D
-P 4600 2500
-F 0 "JP1" H 4600 2705 50  0000 C CNN
-F 1 "SolderJumper_2_Bridged" H 4600 2614 50  0000 C CNN
-F 2 "Jumper:SolderJumper-2_P1.3mm_Bridged2Bar_Pad1.0x1.5mm" H 4600 2500 50  0001 C CNN
-F 3 "~" H 4600 2500 50  0001 C CNN
-	1    4600 2500
-	1    0    0    -1
-$EndComp
-Wire Wire Line
-	4200 2500 4450 2500
 Connection ~ 4200 2500
 $Comp
@@
 Wire Wire Line
 	5000 2750 5000 2500
-Wire Wire Line
-	4750 2500 5000 2500
 $Comp
 L power:VCC #PWR04
@@
 Wire Wire Line
 	9050 4250 9500 4250
+Wire Wire Line
+	4200 2500 5000 2500
 $EndSCHEMATC
