File: arduino_pro_mini.kicad_pcb (KiCad board)
At the start: 2 copper layers, 33.7 x 27.9 mm, 17 parts, among them J1 Conn_02x03_Odd_Even, J2 Conn_01x10, J3 Conn_01x10, SW1 SW_Push, U1 MIC5205-2.5YM5, U2 ATmega328-AU, Y1 16MHZ

Commit message: update berger drill file
Routing:
- net RX: track 20.2 -> 21.1 mm
- net GND: vias 10 -> 11
Changed lines of the file:
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@@
     (thickness 1.6)
     (drawings 8)
-    (tracks 347)
+    (tracks 352)
     (zones 0)
     (modules 17)
@@
   (layers
     (0 F.Cu signal)
-    (31 B.Cu signal hide)
+    (31 B.Cu signal)
     (32 B.Adhes user)
     (33 F.Adhes user)
@@
       (psnegative false)
       (psa4output false)
-      (plotreference true)
-      (plotvalue true)
+      (plotreference false)
+      (plotvalue false)
       (plotinvisibletext false)
       (padsonsilk false)
@@
       (outputformat 1)
       (mirror false)
-      (drillshape 1)
+      (drillshape 0)
       (scaleselection 1)
-      (outputdirectory ""))
+      (outputdirectory "./"))
   )
   (net 0 "")
@@
   (gr_line (start 139.7 33.02) (end 139.7 55.88) (layer Edge.Cuts) (width 0.05))
   (gr_line (start 142.24 30.48) (end 170.815 30.48) (layer Edge.Cuts) (width 0.05))
+  (via (at 145.415 50.165) (size 0.635) (drill 0.3048) (layers F.Cu B.Cu) (net 1))
   (via (at 160.655 57.15) (size 0.635) (drill 0.3048) (layers F.Cu B.Cu) (net 1))
   (via (at 155.575 57.15) (size 0.635) (drill 0.3048) (layers F.Cu B.Cu) (net 1))
@@
   (segment (start 158.435 51.435) (end 161.29 51.435) (width 0.25) (layer F.Cu) (net 2))
   (segment (start 157.48 50.48) (end 158.435 51.435) (width 0.25) (layer F.Cu) (net 2))
-  (segment (start 156.494334 38.562914) (end 155.42099 37.48957) (width 0.25) (layer B.Cu) (net 2))
-  (segment (start 149.792081 36.83) (end 148.59 36.83) (width 0.25) (layer B.Cu) (net 2))
-  (segment (start 156.494334 45.635279) (end 156.494334 38.562914) (width 0.25) (layer B.Cu) (net 2))
-  (segment (start 161.29 51.435) (end 161.29 50.430945) (width 0.25) (layer B.Cu) (net 2))
-  (segment (start 154.524363 37.48957) (end 153.380878 38.633055) (width 0.25) (layer B.Cu) (net 2))
-  (segment (start 155.42099 37.48957) (end 154.524363 37.48957) (width 0.25) (layer B.Cu) (net 2))
-  (segment (start 153.380878 38.633055) (end 151.595136 38.633055) (width 0.25) (layer B.Cu) (net 2))
-  (segment (start 151.595136 38.633055) (end 149.792081 36.83) (width 0.25) (layer B.Cu) (net 2))
-  (segment (start 161.29 50.430945) (end 156.494334 45.635279) (width 0.25) (layer B.Cu) (net 2))
   (segment (start 158.26 48.58) (end 157.48 48.58) (width 0.25) (layer F.Cu) (net 2))
   (segment (start 158.75 49.07) (end 158.26 48.58) (width 0.25) (layer F.Cu) (net 2))
@@
   (segment (start 158.26 50.48) (end 158.75 49.99) (width 0.25) (layer F.Cu) (net 2))
   (segment (start 157.48 50.48) (end 158.26 50.48) (width 0.25) (layer F.Cu) (net 2))
+  (segment (start 149.792081 36.83) (end 148.59 36.83) (width 0.25) (layer B.Cu) (net 2))
+  (segment (start 151.595136 38.633055) (end 149.792081 36.83) (width 0.25) (layer B.Cu) (net 2))
+  (segment (start 153.380878 38.633055) (end 151.595136 38.633055) (width 0.25) (layer B.Cu) (net 2))
+  (segment (start 154.524363 37.48957) (end 153.380878 38.633055) (width 0.25) (layer B.Cu) (net 2))
+  (segment (start 156.445129 38.513709) (end 155.42099 37.48957) (width 0.25) (layer B.Cu) (net 2))
+  (segment (start 161.29 51.435) (end 161.29 50.430945) (width 0.25) (layer B.Cu) (net 2))
+  (segment (start 156.494334 42.759836) (end 156.445129 42.710631) (width 0.25) (layer B.Cu) (net 2))
+  (segment (start 156.494334 45.635279) (end 156.494334 42.759836) (width 0.25) (layer B.Cu) (net 2))
+  (segment (start 156.445129 42.710631) (end 156.445129 38.513709) (width 0.25) (layer B.Cu) (net 2))
+  (segment (start 161.29 50.430945) (end 156.494334 45.635279) (width 0.25) (layer B.Cu) (net 2))
+  (segment (start 155.42099 37.48957) (end 154.524363 37.48957) (width 0.25) (layer B.Cu) (net 2))
   (segment (start 168.91 50.8) (end 168.91 54.61) (width 0.381) (layer F.Cu) (net 3))
   (segment (start 160.145 53.99) (end 160.02 54.115) (width 0.381) (layer F.Cu) (net 3))
@@
   (segment (start 145.705 47.455) (end 145.705 42.255) (width 0.25) (layer F.Cu) (net 8))
   (segment (start 152.78 52.515) (end 153.67 52.515) (width 0.25) (layer F.Cu) (net 8))
-  (segment (start 152.4 55.88) (end 152.4 52.895) (width 0.25) (layer F.Cu) (net 8))
+  (segment (start 152.4 52.895) (end 152.78 52.515) (width 0.25) (layer F.Cu) (net 8))
+  (segment (start 151.194741 57.085259) (end 152.4 55.88) (width 0.25) (layer F.Cu) (net 8))
   (segment (start 147.375259 57.085259) (end 151.194741 57.085259) (width 0.25) (layer F.Cu) (net 8))
   (segment (start 145.815009 55.525009) (end 147.375259 57.085259) (width 0.25) (layer F.Cu) (net 8))
-  (segment (start 151.194741 57.085259) (end 152.4 55.88) (width 0.25) (layer F.Cu) (net 8))
   (segment (start 145.815009 55.304991) (end 145.815009 55.525009) (width 0.25) (layer F.Cu) (net 8))
+  (segment (start 147.32 53.8) (end 145.815009 55.304991) (width 0.25) (layer F.Cu) (net 8))
+  (segment (start 152.4 55.88) (end 152.4 52.895) (width 0.25) (layer F.Cu) (net 8))
   (segment (start 147.32 48.26) (end 147.32 53.8) (width 0.25) (layer F.Cu) (net 8))
   (segment (start 146.515 47.455) (end 147.32 48.26) (width 0.25) (layer F.Cu) (net 8))
-  (segment (start 152.4 52.895) (end 152.78 52.515) (width 0.25) (layer F.Cu) (net 8))
-  (segment (start 147.32 53.8) (end 145.815009 55.304991) (width 0.25) (layer F.Cu) (net 8))
   (segment (start 145.705 47.455) (end 146.515 47.455) (width 0.25) (layer F.Cu) (net 8))
   (via (at 154.305 38.735) (size 0.635) (drill 0.3048) (layers F.Cu B.Cu) (net 9))
@@
   (segment (start 167.64 34.289994) (end 167.004994 34.925) (width 0.25) (layer F.Cu) (net 13))
   (segment (start 167.64 33.02) (end 167.64 34.289994) (width 0.25) (layer F.Cu) (net 13))
-  (segment (start 157.48 37.534498) (end 160.089498 34.925) (width 0.25) (layer B.Cu) (net 13))
-  (segment (start 157.48 43.18) (end 157.48 37.534498) (width 0.25) (layer B.Cu) (net 13))
-  (segment (start 160.089498 34.925) (end 167.004994 34.925) (width 0.25) (layer B.Cu) (net 13))
+  (segment (start 159.402374 34.925) (end 167.004994 34.925) (width 0.25) (layer B.Cu) (net 13))
+  (segment (start 156.845 42.545) (end 156.845 37.482374) (width 0.25) (layer B.Cu) (net 13))
+  (segment (start 156.845 37.482374) (end 159.402374 34.925) (width 0.25) (layer B.Cu) (net 13))
+  (segment (start 157.48 43.18) (end 156.845 42.545) (width 0.25) (layer B.Cu) (net 13))
   (via (at 165.1 35.56) (size 0.635) (drill 0.3048) (layers F.Cu B.Cu) (net 14))
   (segment (start 165.1 33.02) (end 165.1 35.56) (width 0.25) (layer F.Cu) (net 14))
@@
   (via (at 158.696131 41.963869) (size 0.635) (drill 0.3048) (layers F.Cu B.Cu) (net 16))
   (segment (start 159.372262 42.64) (end 158.696131 41.963869) (width 0.25) (layer F.Cu) (net 16))
-  (segment (start 158.115 41.382738) (end 158.696131 41.963869) (width 0.25) (layer B.Cu) (net 16))
-  (segment (start 158.115 39.317125) (end 158.115 41.382738) (width 0.25) (layer B.Cu) (net 16))
-  (segment (start 161.898562 35.533563) (end 158.115 39.317125) (width 0.25) (layer B.Cu) (net 16))
+  (segment (start 158.75 41.91) (end 158.696131 41.963869) (width 0.25) (layer B.Cu) (net 16))
+  (segment (start 158.75 38.735) (end 158.75 41.91) (width 0.25) (layer B.Cu) (net 16))
+  (segment (start 161.898562 35.586438) (end 158.75 38.735) (width 0.25) (layer B.Cu) (net 16))
+  (segment (start 161.898562 35.533563) (end 161.898562 35.586438) (width 0.25) (layer B.Cu) (net 16))
   (segment (start 157.67975 33.02) (end 157.48 33.02) (width 0.25) (layer F.Cu) (net 17))
   (segment (start 159.01 34.55) (end 159.01 36.39) (width 0.25) (layer F.Cu) (net 17))
@@
   (segment (start 149.225 43.18) (end 149.765 42.64) (width 0.25) (layer F.Cu) (net 28))
   (zone (net 1) (net_name GND) (layer F.Cu) (hatch edge 0.508)
-    (connect_pads yes (clearance 0.508))
-    (min_thickness 0.254)
-    (fill yes (arc_segments 32) (thermal_gap 0.508) (thermal_bridge_width 0.508))
-    (polygon
-      (pts
-        (xy 173.355 58.42) (xy 139.7 58.42) (xy 139.7 30.48) (xy 173.355 30.48)
-      )
-    )
-  )
-  (zone (net 1) (net_name GND) (layer B.Cu) (hatch edge 0.508)
-    (connect_pads yes (clearance 0.508))
-    (min_thickness 0.254)
-    (fill yes (arc_segments 32) (thermal_gap 0.508) (thermal_bridge_width 0.508))
-    (polygon
-      (pts
-        (xy 173.355 58.42) (xy 139.7 58.42) (xy 139.7 30.48) (xy 173.355 30.48)
-      )
-    )
-  )
-  (zone (net 1) (net_name GND) (layer B.Cu) (hatch edge 0.508)
     (connect_pads yes (clearance 0.2))
     (min_thickness 0.254)
@@
   )
   (zone (net 1) (net_name GND) (layer B.Cu) (hatch edge 0.508)
-    (connect_pads yes (clearance 0.508))
+    (connect_pads yes (clearance 0.2))
     (min_thickness 0.254)
     (fill yes (arc_segments 32) (thermal_gap 0.508) (thermal_bridge_width 0.508))
